Commit message: Add lidar link and joint

File: src/home_cleaning_robot/urdf/cleaning_bot.urdf (robot description, URDF)
Before this commit: robot cleaning_bot, 5 links, 4 joints
Links:
- added link lidar_link, mass 0.2; collision box size=.5 .5 .5; visual box size=.5 .5 .5
Joints:
- added joint base_lidar_joint: type fixed, parent base_link, child lidar_link, origin xyz=1.75 0 .75 rpy=0.0 0.0 0.0
