Commit message: Switch to xacro

File: src/home_cleaning_robot/urdf/cleaning_bot.xacro (robot description, xacro)
@@ -1,19 +1,22 @@
 <?xml version="1.0"?>
-<robot name="cleaning_bot">
+<robot xmlns:xacro="http://www.ros.org/wiki/xacro" name="cleaning_bot">
+    <!-- Xacro property for color brightness. -->
+    <xacro:property name="bright" value=".75" />
+    <xacro:property name="alpha" value="1" />
     <!-- List of materials for easier viewing. -->
     <material name="red">
-        <color rgba=".75 0.0 0.0 1"/>
+        <color rgba="${bright} 0.0 0.0 ${alpha}"/>
     </material>
     <material name="blue">
-        <color rgba="0 0 .75 1" />
+        <color rgba="0 0 ${bright} ${alpha}" />
     </material>
     <material name="green">
-        <color rgba="0 .75 0 1" />
+        <color rgba="0 ${bright} 0 ${alpha}" />
     </material>
     <material name="white">
-        <color rgba=".75 .75 .75 1"/>
+        <color rgba="${bright} ${bright} ${bright} ${alpha}"/>
     </material>
     <material name="purple">
-        <color rgba=".75 0 1 1" />
+        <color rgba="${bright} 0 ${bright*0.75} ${alpha}" />
     </material>
     <!-- World link as the root. -->

Commit message: Add easy scaling with xacro property

File: src/home_cleaning_robot/urdf/cleaning_bot.xacro (robot description, xacro)
@@ -1,7 +1,16 @@
 <?xml version="1.0"?>
 <robot xmlns:xacro="http://www.ros.org/wiki/xacro" name="cleaning_bot">
-    <!-- Xacro property for color brightness. -->
+    <!-- Xacro property for color brightness and alpha. -->
     <xacro:property name="bright" value=".75" />
     <xacro:property name="alpha" value="1" />
+    <!-- Xacro property for scale. -->
+    <xacro:property name="scale" value="1" />
+    <!-- Scale derived from 'scale' property. -->
+    <xacro:property name="chassis_radius" value="${scale*2}" />
+    <xacro:property name="chassis_length" value="${scale*1}" />
+    <xacro:property name="wheel_radius" value="${chassis_radius/2}" />
+    <xacro:property name="wheel_length" value="${chassis_length/2}" />
+    <xacro:property name="caster_radius" value="${chassis_radius/4}" />
+    <xacro:property name="lidar_length" value="${chassis_radius/4}" />
     <!-- List of materials for easier viewing. -->
     <material name="red">
@@ -26,5 +35,5 @@
         <visual>
            <geometry>
-                <cylinder radius="2.0" length="1.0"/>
+                <cylinder radius="${chassis_radius}" length="${chassis_length}"/>
            </geometry>
            <material name="white"/>
@@ -32,5 +41,5 @@
         <collision>
             <geometry>
-                <cylinder radius="2.0" length="1.0"/>
+                <cylinder radius="${chassis_radius}" length="${chassis_length}"/>
             </geometry>
         </collision>
@@ -44,5 +53,5 @@
         <visual>
             <geometry>
-                <cylinder radius="1.0" length=".5"/>
+                <cylinder radius="${wheel_radius}" length="${wheel_length}"/>
             </geometry>
             <material name="blue"/>
@@ -50,5 +59,5 @@
         <collision>
             <geometry>
-                <cylinder radius="1.0" length=".5"/>
+                <cylinder radius="${wheel_radius}" length="${wheel_length}"/>
             </geometry>
         </collision>
@@ -62,5 +71,5 @@
         <visual>
             <geometry>
-                <cylinder radius="1.0" length=".5"/>
+                <cylinder radius="${wheel_radius}" length="${wheel_length}"/>
             </geometry>
             <material name="red"/>
@@ -68,5 +77,5 @@
         <collision>
             <geometry>
-                <cylinder radius="1.0" length=".5"/>
+                <cylinder radius="${wheel_radius}" length="${wheel_length}"/>
             </geometry>
         </collision>
@@ -80,5 +89,5 @@
         <visual>
             <geometry>
-                <sphere radius=".5"/>
+                <sphere radius="${caster_radius}"/>
             </geometry>
             <material name="green"/>
@@ -86,5 +95,5 @@
         <collision>
             <geometry>
-                <sphere radius="1.0"/>
+                <sphere radius="${caster_radius}"/>
             </geometry>
         </collision>
@@ -98,5 +107,5 @@
         <visual>
             <geometry>
-                <box size=".5 .5 .5"/>
+                <box size="${lidar_length} ${lidar_length} ${lidar_length}"/>
             </geometry>
             <material name="purple"/>
@@ -104,5 +113,5 @@
         <collision>
             <geometry>
-                <box size=".5 .5 .5"/>
+                <box size="${lidar_length} ${lidar_length} ${lidar_length}"/>
             </geometry>
         </collision>
@@ -116,5 +125,5 @@
         <parent link="world"/>
         <child link="base_link"/>
-        <origin xyz="0.0 0.0 1.5" rpy="0.0 0.0 1.57" />
+        <origin xyz="0.0 0.0 ${chassis_radius+caster_radius}" rpy="0.0 0.0 1.57" />
     </joint>
     <!-- This joint defines base/left-wheel joint. -->
@@ -122,5 +131,5 @@
         <parent link="base_link"/>
         <child link="left_wheel_link"/>
-        <origin xyz="0 2.25 -.5" rpy="1.57 0 0"/>
+        <origin xyz="0 ${chassis_radius+wheel_length/2} -${chassis_length/2}" rpy="1.57 0 0"/>
         <axis xyz="0 0 1"/>
     </joint>
@@ -129,5 +138,5 @@
         <parent link="base_link"/>
         <child link="right_wheel_link"/>
-        <origin xyz="0 -2.25 -.5" rpy="1.57 0 0"/>
+        <origin xyz="0 -${chassis_radius+wheel_length/2} -${chassis_length/2}" rpy="1.57 0 0"/>
         <axis xyz="0 0 1"/>
     </joint>
@@ -136,5 +145,5 @@
         <parent link="base_link"/>
         <child link="caster_wheel_link"/>
-        <origin xyz="0 0 -1" rpy="0.0 0.0 0.0"/>
+        <origin xyz="0 0 -${chassis_length}" rpy="0.0 0.0 0.0"/>
     </joint>
     <!-- This joint defines base/lidar joint. -->
@@ -142,5 +151,5 @@
         <parent link="base_link"/>
         <child link="lidar_link"/>
-        <origin xyz="1.75 0 .75" rpy="0.0 0.0 0.0"/>
+        <origin xyz="${chassis_radius-lidar_length/2} 0 ${chassis_length-lidar_length/2}" rpy="0.0 0.0 0.0"/>
     </joint>
 </robot>

Commit message: Fix robot too large

File: src/home_cleaning_robot/urdf/cleaning_bot.xacro (robot description, xacro)
@@ -5,5 +5,5 @@
     <xacro:property name="alpha" value="1" />
     <!-- Xacro property for scale. -->
-    <xacro:property name="scale" value="1" />
+    <xacro:property name="scale" value=".15" />
     <!-- Scale derived from 'scale' property. -->
     <xacro:property name="chassis_radius" value="${scale*2}" />

Commit message: Xacro inertial macro and no longer fixed to world

File: src/home_cleaning_robot/urdf/cleaning_bot.xacro (robot description, xacro)
@@ -13,4 +13,11 @@
     <xacro:property name="caster_radius" value="${chassis_radius/4}" />
     <xacro:property name="lidar_length" value="${chassis_radius/4}" />
+    <!-- Default inertial from ROS tutorials. -->
+    <xacro:macro name="default_inertial" params="mass">
+    <inertial>
+        <mass value="${mass*scale}" />
+        <inertia ixx="1.0" ixy="0.0" ixz="0.0" iyy="1.0" iyz="0.0" izz="1.0" />
+    </inertial>
+    </xacro:macro>
     <!-- List of materials for easier viewing. -->
     <material name="red">
@@ -29,6 +36,4 @@
         <color rgba="${bright} 0 ${bright*0.75} ${alpha}" />
     </material>
-    <!-- World link as the root. -->
-    <link name="world"/>
     <!-- This is the base link of the robot. A simple cylinderical chassis. -->
     <link name="base_link">
@@ -44,8 +49,5 @@
             </geometry>
         </collision>
-        <inertial>
-            <mass value="10.0"/>
-            <inertia ixx="10.8333" ixy="0.0" ixz="0.0" iyy="10.8333" iyz="0.0" izz="20.0"/>
-        </inertial>
+        <xacro:default_inertial mass="10" />
     </link>
     <!-- This is the left wheel link. -->
@@ -62,8 +64,5 @@
             </geometry>
         </collision>
-        <inertial>
-            <mass value="1.0"/>
-            <inertia ixx="0.2708" ixy="0.0" ixz="0.0" iyy="0.2708" iyz="0.0" izz="0.5"/>
-        </inertial>
+        <xacro:default_inertial mass="10" />
     </link>
     <!-- This is the right wheel link. -->
@@ -80,8 +79,5 @@
             </geometry>
         </collision>
-        <inertial>
-            <mass value="1.0"/>
-            <inertia ixx="0.2708" ixy="0.0" ixz="0.0" iyy="0.2708" iyz="0.0" izz="0.5"/>
-        </inertial>
+        <xacro:default_inertial mass="10" />
     </link>
     <!-- The caster wheel. -->
@@ -98,8 +94,5 @@
             </geometry>
         </collision>
-        <inertial>
-            <mass value="0.5"/>
-            <inertia ixx="0.05" ixy="0.0" ixz="0.0" iyy="0.05" iyz="0.0" izz="0.05"/>
-        </inertial>
+        <xacro:default_inertial mass="10" />
     </link>
     <!-- This is the lidar camera link mounted on top of the chassis. -->
@@ -116,15 +109,6 @@
             </geometry>
         </collision>
-        <inertial>
-            <mass value="0.2"/>
-            <inertia ixx="0.004167" ixy="0.0" ixz="0.0" iyy="0.004167" iyz="0.0" izz="0.004167"/>
-        </inertial>
+        <xacro:default_inertial mass="1" />
     </link>
-    <!-- This joint defines offset of base joint from world root. -->
-    <joint name="world_base_joint" type="fixed">
-        <parent link="world"/>
-        <child link="base_link"/>
-        <origin xyz="0.0 0.0 ${chassis_radius+caster_radius}" rpy="0.0 0.0 1.57" />
-    </joint>
     <!-- This joint defines base/left-wheel joint. -->
     <joint name="base_left_wheel_joint" type="continuous">

Commit message: Add gazebo plugins to Xacro

File: src/home_cleaning_robot/urdf/cleaning_bot.xacro (robot description, xacro)
@@ -13,4 +13,5 @@
     <xacro:property name="caster_radius" value="${chassis_radius/4}" />
     <xacro:property name="lidar_length" value="${chassis_radius/4}" />
+    <xacro:property name="wheel_distance" value="${chassis_radius+wheel_length/2}" />
     <!-- Default inertial from ROS tutorials. -->
     <xacro:macro name="default_inertial" params="mass">
@@ -115,6 +116,6 @@
         <parent link="base_link"/>
         <child link="left_wheel_link"/>
-        <origin xyz="0 ${chassis_radius+wheel_length/2} -${chassis_length/2}" rpy="1.57 0 0"/>
-        <axis xyz="0 0 1"/>
+        <origin xyz="0 ${wheel_distance} -${chassis_length/2}" rpy="1.57 0 0"/>
+        <axis xyz="0 0 -1"/>
     </joint>
     <!-- This joint defines base/right-wheel joint. -->
@@ -122,6 +123,6 @@
         <parent link="base_link"/>
         <child link="right_wheel_link"/>
-        <origin xyz="0 -${chassis_radius+wheel_length/2} -${chassis_length/2}" rpy="1.57 0 0"/>
-        <axis xyz="0 0 1"/>
+        <origin xyz="0 -${wheel_distance} -${chassis_length/2}" rpy="1.57 0 0"/>
+        <axis xyz="0 0 -1"/>
     </joint>
     <!-- This joint defines base/caster-wheel joint. -->
@@ -137,3 +138,51 @@
         <origin xyz="${chassis_radius-lidar_length/2} 0 ${chassis_length-lidar_length/2}" rpy="0.0 0.0 0.0"/>
     </joint>
+    <!-- Gazebo LiDAR sensor. -->
+    <gazebo reference="lidar_link">
+        <sensor name="lidar_sensor" type="gpu_lidar">
+            <pose>0 0 0 0 0 0</pose>
+            <update_rate>10</update_rate>
+            <lidar>
+            <scan>
+                <horizontal>
+                <samples>720</samples>
+                <resolution>1</resolution>
+                <min_angle>-1.5708</min_angle>
+                <max_angle>1.5708</max_angle>
+                </horizontal>
+            </scan>
+            <range>
+                <min>0.1</min>
+                <max>30.0</max>
+                <resolution>0.01</resolution>
+            </range>
+            </lidar>
+            <always_on>true</always_on>
+            <visualize>true</visualize>
+            <topic>/scan</topic>
+        </sensor>
+    </gazebo>
+    <!-- Gazebo plugin for diff-drive. Allows the robot to move. -->
+    <gazebo>
+        <plugin filename="gz-sim-diff-drive-system" name="gz::sim::systems::DiffDrive">
+            <!-- Wheel joints -->
+            <left_joint>base_left_wheel_joint</left_joint>
+            <right_joint>base_right_wheel_joint</right_joint>
+            <!-- Robot kinematics -->
+            <wheel_separation>${wheel_distance*2}</wheel_separation>
+            <wheel_radius>${wheel_radius}</wheel_radius>
+            <!-- Motion limits -->
+            <max_linear_velocity>1.0</max_linear_velocity>
+            <max_angular_velocity>2.0</max_angular_velocity>
+            <!-- Command & odometry -->
+            <topic>/cmd_vel</topic>
+            <odom_topic>/odom</odom_topic>
+            <frame_id>odom</frame_id>
+            <child_frame_id>base_link</child_frame_id>
+            <!-- Behavior -->
+            <update_rate>50</update_rate>
+            <publish_odom>true</publish_odom>
+            <publish_tf>true</publish_tf>
+        </plugin>
+    </gazebo>
 </robot>

Commit message: Lidar view düzeltildi

File: src/home_cleaning_robot/urdf/cleaning_bot.xacro (robot description, xacro)
@@ -1,4 +1,4 @@
 <?xml version="1.0"?>
-<robot xmlns:xacro="http://www.ros.org/wiki/xacro" name="cleaning_bot">
+<robot xmlns:xacro="http://www.ros.org/wiki/xacro" xmlns:gz="http://gazebosim.org/schema" name="cleaning_bot">
     <!-- Xacro property for color brightness and alpha. -->
     <xacro:property name="bright" value=".75" />
@@ -105,10 +105,5 @@
             <material name="purple"/>
         </visual>
-        <collision>
-            <geometry>
-                <box size="${lidar_length} ${lidar_length} ${lidar_length}"/>
-            </geometry>
-        </collision>
-        <xacro:default_inertial mass="1" />
+        <xacro:default_inertial mass="0.1" />
     </link>
     <!-- This joint defines base/left-wheel joint. -->
@@ -158,5 +153,5 @@
             </scan>
             <range>
-                <min>0.1</min>
+                <min>0.12</min>
                 <max>30.0</max>
                 <resolution>0.01</resolution>
@@ -165,4 +160,5 @@
             <always_on>true</always_on>
             <visualize>true</visualize>
+            <gz:frame_id>lidar_link</gz:frame_id>
             <topic>/scan</topic>
         </sensor>
@@ -170,4 +166,9 @@
     <!-- Gazebo plugin for diff-drive. Allows the robot to move. -->
     <gazebo>
+    	<plugin filename="libgz-sim-joint-state-publisher-system.so" name="gz::sim::systems::JointStatePublisher">
+            <topic>joint_states</topic>
+            <joint_name>base_left_wheel_joint</joint_name>
+            <joint_name>base_right_wheel_joint</joint_name>
+        </plugin>
         <plugin filename="gz-sim-diff-drive-system" name="gz::sim::systems::DiffDrive">
             <!-- Wheel joints -->

Commit message: stabilize model

File: src/home_cleaning_robot/urdf/cleaning_bot.xacro (robot description, xacro)
@@ -14,4 +14,42 @@
     <xacro:property name="lidar_length" value="${chassis_radius/4}" />
     <xacro:property name="wheel_distance" value="${chassis_radius+wheel_length/2}" />
+    <xacro:property name="caster_distance" value="${chassis_radius * 1.5}" />
+    <!-- Inertial macros with proper tensor calculations. -->
+    <!-- Cylindrical inertia (for chassis) -->
+    <xacro:macro name="cylinder_inertial" params="mass radius length">
+    <inertial>
+        <mass value="${mass}" />
+        <!-- Ixx = Iyy = (1/12)*m*(3*r^2 + h^2), Izz = (1/2)*m*r^2 -->
+        <inertia ixx="${mass*(3*radius*radius + length*length)/12}"
+                 ixy="0.0" ixz="0.0"
+                 iyy="${mass*(3*radius*radius + length*length)/12}"
+                 iyz="0.0"
+                 izz="${mass*radius*radius/2}" />
+    </inertial>
+    </xacro:macro>
+    <!-- Sphere inertial (for caster wheel) -->
+    <xacro:macro name="sphere_inertial" params="mass radius">
+    <inertial>
+        <mass value="${mass}" />
+        <!-- I = (2/5)*m*r^2 for all axes -->
+        <inertia ixx="${mass*radius*radius*2/5}"
+                 ixy="0.0" ixz="0.0"
+                 iyy="${mass*radius*radius*2/5}"
+                 iyz="0.0"
+                 izz="${mass*radius*radius*2/5}" />
+    </inertial>
+    </xacro:macro>
+    <!-- Box inertial (for lidar) -->
+    <xacro:macro name="box_inertial" params="mass length width height">
+    <inertial>
+        <mass value="${mass}" />
+        <!-- Ixx = (1/12)*m*(w^2 + h^2), Iyy = (1/12)*m*(l^2 + h^2), Izz = (1/12)*m*(l^2 + w^2) -->
+        <inertia ixx="${mass*(width*width + height*height)/12}"
+                 ixy="0.0" ixz="0.0"
+                 iyy="${mass*(length*length + height*height)/12}"
+                 iyz="0.0"
+                 izz="${mass*(length*length + width*width)/12}" />
+    </inertial>
+    </xacro:macro>
     <!-- Default inertial from ROS tutorials. -->
     <xacro:macro name="default_inertial" params="mass">
@@ -36,4 +74,7 @@
     <material name="purple">
         <color rgba="${bright} 0 ${bright*0.75} ${alpha}" />
+    </material>
+    <material name="yellow">
+        <color rgba="${bright} ${bright} 0.0 ${alpha}"/>
     </material>
     <!-- This is the base link of the robot. A simple cylinderical chassis. -->
@@ -50,5 +91,5 @@
             </geometry>
         </collision>
-        <xacro:default_inertial mass="10" />
+        <xacro:cylinder_inertial mass="3.0" radius="${chassis_radius}" length="${chassis_length}" />
     </link>
     <!-- This is the left wheel link. -->
@@ -65,5 +106,5 @@
             </geometry>
         </collision>
-        <xacro:default_inertial mass="10" />
+        <xacro:cylinder_inertial mass="1.0" radius="${wheel_radius}" length="${wheel_length}" />
     </link>
     <!-- This is the right wheel link. -->
@@ -80,5 +121,5 @@
             </geometry>
         </collision>
-        <xacro:default_inertial mass="10" />
+        <xacro:cylinder_inertial mass="1.0" radius="${wheel_radius}" length="${wheel_length}" />
     </link>
     <!-- The caster wheel. -->
@@ -95,5 +136,35 @@
             </geometry>
         </collision>
-        <xacro:default_inertial mass="10" />
+        <xacro:sphere_inertial mass="0.5" radius="${caster_radius}" />
+    </link>
+    <!-- The front stabilizer. -->
+    <link name="front_stabilizer_link">
+        <visual>
+            <geometry>
+                <sphere radius="${caster_radius}"/>
+            </geometry>
+            <material name="yellow"/>
+        </visual>
+        <collision>
+            <geometry>
+                <sphere radius="${caster_radius}"/>
+            </geometry>
+        </collision>
+        <xacro:sphere_inertial mass="0.5" radius="${caster_radius}" />
+    </link>
+    <!-- The back stabilizer. -->
+    <link name="back_stabilizer_link">
+        <visual>
+            <geometry>
+                <sphere radius="${caster_radius}"/>
+            </geometry>
+            <material name="yellow"/>
+        </visual>
+        <collision>
+            <geometry>
+                <sphere radius="${caster_radius}"/>
+            </geometry>
+        </collision>
+        <xacro:sphere_inertial mass="0.5" radius="${caster_radius}" />
     </link>
     <!-- This is the lidar camera link mounted on top of the chassis. -->
@@ -105,5 +176,5 @@
             <material name="purple"/>
         </visual>
-        <xacro:default_inertial mass="0.1" />
+        <xacro:box_inertial mass="0.05" length="${lidar_length}" width="${lidar_length}" height="${lidar_length}" />
     </link>
     <!-- This joint defines base/left-wheel joint. -->
@@ -113,4 +184,5 @@
         <origin xyz="0 ${wheel_distance} -${chassis_length/2}" rpy="1.57 0 0"/>
         <axis xyz="0 0 -1"/>
+        <dynamics damping="0.5" friction="0.1"/>
     </joint>
     <!-- This joint defines base/right-wheel joint. -->
@@ -120,4 +192,5 @@
         <origin xyz="0 -${wheel_distance} -${chassis_length/2}" rpy="1.57 0 0"/>
         <axis xyz="0 0 -1"/>
+        <dynamics damping="0.5" friction="0.1"/>
     </joint>
     <!-- This joint defines base/caster-wheel joint. -->
@@ -127,4 +200,14 @@
         <origin xyz="0 0 -${chassis_length}" rpy="0.0 0.0 0.0"/>
     </joint>
+    <joint name="base_front_stabilizer_joint" type="fixed">
+        <parent link="base_link"/>
+        <child link="front_stabilizer_link"/>
+        <origin xyz="${chassis_radius-caster_radius/2} 0 -${chassis_length}" rpy="0.0 0.0 0.0"/>
+    </joint>
+    <joint name="base_back_stabilizer_joint" type="fixed">
+        <parent link="base_link"/>
+        <child link="back_stabilizer_link"/>
+        <origin xyz="-${chassis_radius-caster_radius/2} 0 -${chassis_length}" rpy="0.0 0.0 0.0"/>
+    </joint>
     <!-- This joint defines base/lidar joint. -->
     <joint name="base_lidar_joint" type="fixed">
@@ -133,8 +216,24 @@
         <origin xyz="${chassis_radius-lidar_length/2} 0 ${chassis_length-lidar_length/2}" rpy="0.0 0.0 0.0"/>
     </joint>
-    <gazebo>
-        <plugin filename="gz-sim-sensors-system" name="gz::sim::systems::Sensors">
-            <render_engine>ogre2</render_engine>
-        </plugin>
+    <gazebo reference="base_link">
+        <material>Gazebo/White</material>
+    </gazebo>
+    <gazebo reference="left_wheel_link">
+        <material>Gazebo/Blue</material>
+    </gazebo>
+    <gazebo reference="right_wheel_link">
+        <material>Gazebo/Red</material>
+    </gazebo>
+    <gazebo reference="caster_wheel_link">
+        <material>Gazebo/Green</material>
+    </gazebo>
+    <gazebo reference="left_stabilizer_link">
+        <material>Gazebo/Yellow</material>
+    </gazebo>
+    <gazebo reference="right_stabilizer_link">
+        <material>Gazebo/Yellow</material>
+    </gazebo>
+    <gazebo reference="lidar_link">
+        <material>Gazebo/Purple</material>
     </gazebo>
     <!-- Gazebo LiDAR sensor. -->
@@ -166,4 +265,7 @@
     <!-- Gazebo plugin for diff-drive. Allows the robot to move. -->
     <gazebo>
+        <plugin filename="gz-sim-sensors-system" name="gz::sim::systems::Sensors">
+            <render_engine>ogre2</render_engine>
+        </plugin>
     	<plugin filename="libgz-sim-joint-state-publisher-system.so" name="gz::sim::systems::JointStatePublisher">
             <topic>joint_states</topic>
